Commit message: update assets

File: assets/urdf/robot_without_gripper.urdf (robot description, URDF)
Before this commit: robot ur10e_cell, 18 links, 16 joints
Links:
- added link cylinder_link, mass 0.2; collision cylinder length=0.1 radius=0.01; visual cylinder length=0.1 radius=0.01
- added link tcp_link
Joints:
- added joint cylinder-tcp: type fixed, parent cylinder_link, child tcp_link, origin xyz=0.0 0.0 0.2 rpy=0 0 0
- added joint flange-tool0: type fixed, parent flange, child tool0, origin xyz=0 0 0 rpy=1.5707963267948966 0 1.5707963267948966
- added joint tool1: type fixed, parent tool0, child cylinder_link, origin xyz=0.0 0.0 0.0 rpy=0 0 3.141592653589793

Commit message: added inertials

File: assets/urdf/robot_without_gripper.urdf (robot description, URDF)
Before this commit: robot ur10e_cell, 20 links, 19 joints
Links:
- link base: mass None -> 1.0
- link base_link: mass None -> 1.0
- link corrected_world: mass None -> 1.0
- link flange: mass None -> 1.0
- link ft_frame: mass None -> 1.0
- link platform_link: mass None -> 1
- link tcp_link: mass None -> 1.0
- link tool0: mass None -> 1.0
- link warehouse_link: mass None -> 1
